Commit message: simple poles example

File: drake/poles.urdf (robot description, URDF)
Before this commit: robot holodeck, 2 links, 1 joints
Links:
- added link pole2, mass .5; collision box size=0.042 0.042 3; visual box size=0.042 0.042 3
- added link pole3, mass .5; collision box size=0.042 0.042 3; visual box size=0.042 0.042 3
- link pole1: geometry collision box size=0.042 0.042 3; visual box size=0.042 0.042 3
Joints:
- added joint pole2_weld: type fixed, parent world, child pole2, origin xyz=.9 -.2 0 rpy=0 0 0
- added joint pole3_weld: type fixed, parent world, child pole3, origin xyz=1.1 0 0 rpy=0 0 0

Commit message: working pole trajectory

File: drake/poles.urdf (robot description, URDF)
Before this commit: robot poles, 4 links, 3 joints
Joints:
- joint pole1_weld: origin xyz=.7 .3 0 rpy=0 0 0 -> xyz=.7 .5 0 rpy=0 0 0
- joint pole2_weld: origin xyz=.9 -.2 0 rpy=0 0 0 -> xyz=.9 -.5 0 rpy=0 0 0
- joint pole3_weld: origin xyz=1.1 0 0 rpy=0 0 0 -> xyz=1.4 0 0 rpy=0 0 0
