Commit message: mostly the TILQR at the end and beginning of TVLQR

File: matlab/poles.urdf (robot description, URDF)
Before this commit: robot poles, 4 links, 3 joints
Joints:
- joint pole1_weld: origin xyz=.7 .5 0 rpy=0 0 0 -> xyz=-1 .5 0 rpy=0 0 0
- joint pole2_weld: origin xyz=.9 -.5 0 rpy=0 0 0 -> xyz=-.8 -.5 0 rpy=0 0 0
- joint pole3_weld: origin xyz=1.4 0 0 rpy=0 0 0 -> xyz=-.3 0 0 rpy=0 0 0

Commit message: tvlqr tracking data

File: matlab/poles.urdf (robot description, URDF)
Before this commit: robot poles, 4 links, 3 joints
Joints:
- joint pole1_weld: origin xyz=-1 .5 0 rpy=0 0 0 -> xyz=-.5 .5 0 rpy=0 0 0
- joint pole2_weld: origin xyz=-.8 -.5 0 rpy=0 0 0 -> xyz=-.5 -.5 0 rpy=0 0 0
- joint pole3_weld: origin xyz=-.3 0 0 rpy=0 0 0 -> xyz=0 0 0 rpy=0 0 0
