Commit message: simulation of the kalman filter with vicon dropouts

File: matlab/gates.urdf (robot description, URDF)
Before this commit: robot gates, 13 links, 12 joints
Links:
- removed link h2
- link d1: geometry collision box size=0.042 0.042 1.2; visual box size=0.042 0.042 1.2
- link d2: geometry collision box size=0.042 0.042 1.2; visual box size=0.042 0.042 1.2
- link d3: geometry collision box size=0.042 0.042 1.2; visual box size=0.042 0.042 1.2
- link d4: geometry collision box size=0.042 0.042 1.2; visual box size=0.042 0.042 1.2
- link h1: geometry collision box size=0.042 0.042 1.2; visual box size=0.042 0.042 1.2
Joints:
- removed joint h2_weld
- joint d1_weld: origin xyz=0 .021 1.271 rpy=-1.047197551196598 0 0 -> xyz=0.042 0 1.25 rpy=-1.047197551196598 0 0
- joint d2_weld: origin xyz=0 .021 1.229 rpy=-2.094395102393196 0 0 -> xyz=0.042 0 1.25 rpy=-2.094395102393196 0 0
- joint d3_weld: origin xyz=0 -.021 1.271 rpy=1.047197551196598 0 0 -> xyz=0.042 0 1.25 rpy=1.047197551196598 0 0
- joint d4_weld: origin xyz=0 -.021 1.229 rpy=2.094395102393196 0 0 -> xyz=0.042 0 1.25 rpy=2.094395102393196 0 0
- joint h1_weld: origin xyz=0 -0.021 1.4 rpy=1.570796326794897 0 0 -> xyz=0.042 .1 1.25 rpy=1.570796326794897 0 0
- joint v1_weld: origin xyz=.5 .5 0 rpy=0 0 0 -> xyz=-.5 .5 0 rpy=0 0 0
- joint v2_weld: origin xyz=.5 -.5 0 rpy=0 0 0 -> xyz=-.5 -.5 0 rpy=0 0 0
- joint v3_weld: origin xyz=1 .5 0 rpy=0 0 0 -> xyz=0 .5 0 rpy=0 0 0
- joint v4_weld: origin xyz=1 -.5 0 rpy=0 0 0 -> xyz=0 -.5 0 rpy=0 0 0
- joint v5_weld: origin xyz=1.5 .5 0 rpy=0 0 0 -> xyz=.5 .5 0 rpy=0 0 0
- joint v6_weld: origin xyz=1.5 -.5 0 rpy=0 0 0 -> xyz=.5 -.5 0 rpy=0 0 0

Commit message: compare script

File: matlab/gates.urdf (robot description, URDF)
Before this commit: robot gates, 12 links, 11 joints
Links:
- removed link d1
- removed link d2
- removed link d3
- removed link d4
- removed link h1
- removed link v1
- removed link v2
- removed link v3
- removed link v4
- removed link v5
- removed link v6
- added link l1, mass .5; collision box size=0.042 0.042 3; visual box size=0.042 0.042 3
- added link l2, mass .5; collision box size=0.042 0.042 3; visual box size=0.042 0.042 3
- added link l3, mass .5; collision box size=0.042 0.042 3; visual box size=0.042 0.042 3
- added link l4, mass .5; collision box size=0.042 0.042 3; visual box size=0.042 0.042 3
- added link l5, mass .5; collision box size=0.042 0.042 3; visual box size=0.042 0.042 3
- added link l6, mass .5; collision box size=0.042 0.042 3; visual box size=0.042 0.042 3
- added link s1, mass .5; collision box size=0.042 0.042 1.2; visual box size=0.042 0.042 1.2
- added link s2, mass .5; collision box size=0.042 0.042 1.2; visual box size=0.042 0.042 1.2
- added link s3, mass .5; collision box size=0.042 0.042 1.2; visual box size=0.042 0.042 1.2
- added link s4, mass .5; collision box size=0.042 0.042 1.2; visual box size=0.042 0.042 1.2
- added link s5, mass .5; collision box size=0.042 0.042 1.2; visual box size=0.042 0.042 1.2
Joints:
- removed joint d1_weld
- removed joint d2_weld
- removed joint d3_weld
- removed joint d4_weld
- removed joint h1_weld
- removed joint v1_weld
- removed joint v2_weld
- removed joint v3_weld
- removed joint v4_weld
- removed joint v5_weld
- removed joint v6_weld
- added joint l1_weld: type fixed, parent world, child l1, origin xyz=-.5 .5 0 rpy=0 0 0
- added joint l2_weld: type fixed, parent world, child l2, origin xyz=-.5 -.5 0 rpy=0 0 0
- added joint l3_weld: type fixed, parent world, child l3, origin xyz=0 .5 0 rpy=0 0 0
- added joint l4_weld: type fixed, parent world, child l4, origin xyz=0 -.5 0 rpy=0 0 0
- added joint l5_weld: type fixed, parent world, child l5, origin xyz=.5 .5 0 rpy=0 0 0
- added joint l6_weld: type fixed, parent world, child l6, origin xyz=.5 -.5 0 rpy=0 0 0
- added joint s1_weld: type fixed, parent l2, child s1, origin xyz=0.042 0 1.25 rpy=-1.047197551196598 0 0
- added joint s2_weld: type fixed, parent l2, child s2, origin xyz=0.042 0 1.25 rpy=-2.094395102393196 0 0
- added joint s3_weld: type fixed, parent l3, child s3, origin xyz=0.042 0 1.25 rpy=1.047197551196598 0 0
- added joint s4_weld: type fixed, parent l3, child s4, origin xyz=0.042 0 1.25 rpy=2.094395102393196 0 0
- added joint s5_weld: type fixed, parent l5, child s5, origin xyz=0.042 .1 1.25 rpy=1.570796326794897 0 0

Commit message: working tvlqr with obstacles

File: matlab/gates.urdf (robot description, URDF)
Before this commit: robot gates, 12 links, 11 joints
Links:
- added link m1, mass .5; collision box size=0.042 0.042 1.55; visual box size=0.042 0.042 1.55
Joints:
- added joint m1_weld: type fixed, parent world, child m1, origin xyz=0 0 0 rpy=0 0 0

Commit message: hover button

File: matlab/gates.urdf (robot description, URDF)
Before this commit: robot gates, 13 links, 12 joints
Links:
- removed link m1
Joints:
- removed joint m1_weld
