Commit message: working sysid by modeling the control feedback in the plant

File: matlab/walls.urdf (robot description, URDF)
Before this commit: robot gates2, 14 links, 13 joints
Links:
- removed link l7
- removed link l8
- removed link s1
- removed link s2
- removed link s3
- removed link s4
- removed link s5
- added link wall1, mass .5; collision box size=.01 1 1.5; visual box size=.01 1 1.5
- added link wall2, mass .5; collision box size=.01 .7 3; visual box size=.01 .7 3
- added link wall3, mass .5; collision box size=.01 1 1.5; visual box size=.01 1 1.5
Joints:
- removed joint l7_weld
- removed joint l8_weld
- removed joint s1_weld
- removed joint s2_weld
- removed joint s3_weld
- removed joint s4_weld
- removed joint s5_weld
- added joint wall1_weld: type fixed, parent world, child wall1, origin xyz=-.5 0 0 rpy=0 0 0
- added joint wall2_weld: type fixed, parent world, child wall2, origin xyz=0 -.15 0 rpy=0 0 0
- added joint wall3_weld: type fixed, parent world, child wall3, origin xyz=.5 0 1 rpy=0 0 0
