Commit message: some sysid and the final trajectories

File: matlab/pipes.urdf (robot description, URDF)
Before this commit: robot pipes, 13 links, 12 joints
Links:
- link m1: geometry collision box size=0.042 0.042 1.5; visual box size=0.042 0.042 1.5

File: matlab/walls.urdf (robot description, URDF)
Before this commit: robot walls, 10 links, 9 joints
Links:
- removed link wall3
- added link l7, mass .5; collision box size=0.042 0.042 3; visual box size=0.042 0.042 3
- added link l8, mass .5; collision box size=0.042 0.042 3; visual box size=0.042 0.042 3
- link wall2: geometry collision box size=.01 1 1.5; visual box size=.01 1 1.5
Joints:
- removed joint wall3_weld
- added joint l7_weld: type fixed, parent world, child l7, origin xyz=-.25 0 0 rpy=0 0 0
- added joint l8_weld: type fixed, parent world, child l8, origin xyz=.25 0 0 rpy=0 0 0
- joint wall1_weld: origin xyz=-.5 0 0 rpy=0 0 0 -> xyz=-.5 0 .25 rpy=0 0 0
- joint wall2_weld: origin xyz=0 -.15 0 rpy=0 0 0 -> xyz=.5 0 1 rpy=0 0 0

Commit message: ploting files and modeling

File: matlab/pipes.urdf (robot description, URDF)
Before this commit: robot pipes, 13 links, 12 joints
Links:
- removed link s5
- added link l7, mass .5; collision box size=0.042 0.042 3; visual box size=0.042 0.042 3
Joints:
- removed joint s5_weld
- added joint l7_weld: type fixed, parent world, child l7, origin xyz=.5 -.25 0 rpy=0 0 0

File: matlab/walls.urdf (robot description, URDF)
Before this commit: robot walls, 11 links, 10 joints
Links:
- removed link l8
Joints:
- removed joint l8_weld
- joint l7_weld: origin xyz=-.25 0 0 rpy=0 0 0 -> xyz=0 0 0 rpy=0 0 0
